Commit message: Updated description so that simulation doesn't bounce
Thanks to Kyrre for suggesting changes to PID control parameters!

File: dyret_description/urdf/body.urdf.xacro (robot description, xacro)
@@ -23,5 +23,5 @@
 				</geometry>
 			</collision>
-			<xacro:box_inertia mass="0.58" width="${body_width}"
+			<xacro:box_inertia mass="0.2" width="${body_width}"
 				length="${body_depth}" height="${body_height}"
 				r="${pi/2}" />
@@ -45,5 +45,5 @@
 				</geometry>
 			</collision>
-			<xacro:box_inertia mass="0.28" width="${ac_width}"
+			<xacro:box_inertia mass="0.12" width="${ac_width}"
 				length="${ac_depth}" height="${ac_height}"
 				r="${pi/2}" />

File: dyret_description/urdf/dyret.xacro (robot description, xacro)
@@ -12,7 +12,7 @@
 		<plugin name="controller" filename="libdyret_gazebo_plugin.so">
 			<updateRate>50</updateRate>
-			<pid>100 0 0</pid>
-			<pid type="mx64">86 0 10</pid>
-			<pid type="mx106">32 0 10</pid>
+			<pid>1.0 0 0</pid>
+			<pid type="mx64">8.6 0 1.0</pid>
+			<pid type="mx106">3.2 0 1.0</pid>
 		</plugin>
 	</gazebo>

File: dyret_description/urdf/joints/foot.urdf.xacro (robot description, xacro)
@@ -38,4 +38,10 @@
 		<xacro:if value="$(arg contact_enabled)">
 			<gazebo reference="${name}_foot_sph">
+				<kp>1000000.0</kp>
+				<kd>100.0</kd>
+				<mu1>1.5</mu1>
+				<mu2>1.5</mu2>
+				<maxVel>1.0</maxVel>
+				<minDepth>0.0</minDepth>
 				<sensor name="${name}_bumper" type="contact">
 					<contact>
@@ -51,4 +57,22 @@
 			</gazebo>
 		</xacro:if>
+		<xacro:unless value="$(arg contact_enabled)">
+			<gazebo reference="${name}_foot_sph">
+				<kp>1000000.0</kp>
+				<kd>100.0</kd>
+				<mu1>1.5</mu1>
+				<mu2>1.5</mu2>
+				<maxVel>1.0</maxVel>
+				<minDepth>0.0</minDepth>
+			</gazebo>
+		</xacro:unless>
+		<gazebo reference="${name}_foot_cyl">
+			<kp>1000000.0</kp>
+			<kd>100.0</kd>
+			<mu1>1.5</mu1>
+			<mu2>1.5</mu2>
+			<maxVel>1.0</maxVel>
+			<minDepth>0.0</minDepth>
+		</gazebo>
 	</xacro:macro>
 </robot>

File: dyret_description/urdf/joints/large_extend.urdf.xacro (robot description, xacro)
@@ -57,5 +57,9 @@
 				lower="-0.100" upper="0.0"
 				effort="100.0" velocity="0.00045" />
+			<dynamics damping="1" friction="0.1" />
 		</joint>
+		<gazebo reference="${name}">
+			<implicitSpringDamper>1</implicitSpringDamper>
+		</gazebo>
 	</xacro:macro>
 </robot>

File: dyret_description/urdf/joints/mx106.urdf.xacro (robot description, xacro)
@@ -112,5 +112,4 @@
 			<parent link="${name}_bracket" />
 			<child link="${name}_servo" />
-			<origin xyz="0 0 0" />
 			<limit
 				lower="-1.9" upper="1.9"
@@ -118,4 +117,7 @@
 			<dynamics friction="0.1" damping="0.0952" />
 		</joint>
+		<gazebo reference="${name}">
+			<implicitSpringDamper>1</implicitSpringDamper>
+		</gazebo>
 	</xacro:macro>
 	<xacro:macro name="mx106t_fr08h101_inv" params="name">
@@ -131,4 +133,7 @@
 			<dynamics friction="0.1" damping="0.0952" />
 		</joint>
+		<gazebo reference="${name}">
+			<implicitSpringDamper>1</implicitSpringDamper>
+		</gazebo>
 	</xacro:macro>
 </robot>

File: dyret_description/urdf/joints/mx64at.urdf.xacro (robot description, xacro)
@@ -72,4 +72,7 @@
 			<dynamics friction="0.1" damping="0.0952" />
 		</joint>
+		<gazebo reference="${name}">
+			<implicitSpringDamper>1</implicitSpringDamper>
+		</gazebo>
 	</xacro:macro>
 </robot>

File: dyret_description/urdf/joints/small_extend.urdf.xacro (robot description, xacro)
@@ -57,5 +57,9 @@
 				lower="-0.025" upper="0.0"
 				effort="100.0" velocity="0.00045" />
+			<dynamics damping="1" friction="0.1" />
 		</joint>
+		<gazebo reference="${name}">
+			<implicitSpringDamper>1</implicitSpringDamper>
+		</gazebo>
 	</xacro:macro>
 </robot>
