Commit message: Added contact sensors

File: dyret_description/urdf/dyret.xacro (robot description, xacro)
@@ -2,5 +2,5 @@
 <robot name="dyret" xmlns:xacro="http://ros.org/wiki/xacro">
 	<!-- Arguments that can be passed to this URDF file: -->
-	<xacro:arg name="imu_enabled" default="false" />
+	<xacro:arg name="imu_enabled" default="true" />
 	<xacro:arg name="contact_enabled" default="false" />
 	<!-- Import actual robot and instantiate: -->
@@ -10,7 +10,4 @@
 	<gazebo>
 		<self_collide>true</self_collide>
-		<plugin name="gazebo_ros_control" filename="libgazebo_ros_control.so">
-			<robotNamespace>/dyret</robotNamespace>
-		</plugin>
 	</gazebo>
 </robot>

File: dyret_description/urdf/imu.urdf.xacro (robot description, xacro)
@@ -33,8 +33,9 @@
 					<plugin filename="libgazebo_ros_imu_sensor.so" name="imu_plugin">
 						<bodyName>imu_link</bodyName>
-						<frameName>dyret_body</frameName>
+						<frameName>world</frameName>
 						<gaussianNoise>0.05</gaussianNoise>
+						<robotNamespace>/dyret</robotNamespace>
 						<rpyOffset>0 0 0</rpyOffset>
-						<topicName>dyret/imu</topicName>
+						<topicName>imu</topicName>
 						<updateRateHZ>100.0</updateRateHZ>
 						<xyzOffset>0 0 0</xyzOffset>

File: dyret_description/urdf/joints/foot.urdf.xacro (robot description, xacro)
@@ -36,4 +36,19 @@
 			<origin xyz="0 0 ${-0.0355/2 + 0.00195}" />
 		</joint>
+		<xacro:if value="$(arg contact_enabled)">
+			<gazebo reference="${name}_foot_sph">
+				<sensor name="${name}_bumper" type="contact">
+					<contact>
+						<collision>${name}_ext2_outer_fixed_joint_lump__${name}_foot_sph_collision_2</collision>
+					</contact>
+					<plugin name="${name}_gazebo_ros_bumper_controller"
+						filename="libgazebo_ros_bumper.so">
+						<robotNamespace>/dyret</robotNamespace>
+						<bumperTopicName>${name}_contact</bumperTopicName>
+						<frameName>world</frameName>
+					</plugin>
+				</sensor>
+			</gazebo>
+		</xacro:if>
 	</xacro:macro>
 </robot>

File: dyret_description/urdf/leg.urdf.xacro (robot description, xacro)
@@ -41,4 +41,19 @@
 			<origin xyz="0 0 ${-large_ext2_height - 0.0355/2}" />
 		</joint>
+		<xacro:if value="$(arg contact_enabled)">
+			<gazebo reference="${name}_foot_sph">
+				<sensor name="${name}_bumper" type="contact">
+					<contact>
+						<collision>${name}_foot_sph_collision</collision>
+					</contact>
+					<plugin name="${name}_gazebo_ros_bumper_controller"
+						filename="libgazebo_ros_bumper.so">
+						<robotNamespace>/dyret</robotNamespace>
+						<bumperTopicName>${name}_contact</bumperTopicName>
+						<frameName>world</frameName>
+					</plugin>
+				</sensor>
+			</gazebo>
+		</xacro:if>
 	</xacro:macro>
 </robot>

Commit message: Added Gazebo Plugin for Dyret

File: dyret_description/urdf/dyret.xacro (robot description, xacro)
@@ -10,4 +10,8 @@
 	<gazebo>
 		<self_collide>true</self_collide>
+		<plugin name="controller" filename="libdyret_gazebo_plugin.so">
+			<updateRate>60</updateRate>
+			<pid>48 0 0</pid>
+		</plugin>
 	</gazebo>
 </robot>

File: dyret_description/urdf/leg.urdf.xacro (robot description, xacro)
@@ -41,19 +41,4 @@
 			<origin xyz="0 0 ${-large_ext2_height - 0.0355/2}" />
 		</joint>
-		<xacro:if value="$(arg contact_enabled)">
-			<gazebo reference="${name}_foot_sph">
-				<sensor name="${name}_bumper" type="contact">
-					<contact>
-						<collision>${name}_foot_sph_collision</collision>
-					</contact>
-					<plugin name="${name}_gazebo_ros_bumper_controller"
-						filename="libgazebo_ros_bumper.so">
-						<robotNamespace>/dyret</robotNamespace>
-						<bumperTopicName>${name}_contact</bumperTopicName>
-						<frameName>world</frameName>
-					</plugin>
-				</sensor>
-			</gazebo>
-		</xacro:if>
 	</xacro:macro>
 </robot>

Commit message: Updated default PIDs for extension joints

File: dyret_description/urdf/dyret.xacro (robot description, xacro)
@@ -12,7 +12,7 @@
 		<plugin name="controller" filename="libdyret_gazebo_plugin.so">
 			<updateRate>50</updateRate>
-			<pid>1.0 0 0</pid>
-			<pid type="mx64">8.6 0 1.0</pid>
-			<pid type="mx106">3.2 0 1.0</pid>
+			<pid>1000.0 0.0 0</pid>
+			<pid type="mx64">8.6 0.5 1.0</pid>
+			<pid type="mx106">3.2 0.5 1.0</pid>
 		</plugin>
 	</gazebo>

File: dyret_description/urdf/joints/large_extend.urdf.xacro (robot description, xacro)
@@ -57,5 +57,5 @@
 				lower="-0.100" upper="0.0"
 				effort="100.0" velocity="0.00045" />
-			<dynamics damping="1" friction="0.1" />
+			<!--<dynamics damping="0.7" friction="0.1" />-->
 		</joint>
 		<gazebo reference="${name}">

File: dyret_description/urdf/joints/small_extend.urdf.xacro (robot description, xacro)
@@ -57,5 +57,5 @@
 				lower="-0.025" upper="0.0"
 				effort="100.0" velocity="0.00045" />
-			<dynamics damping="1" friction="0.1" />
+			<dynamics damping="0.7" friction="0.1" />
 		</joint>
 		<gazebo reference="${name}">

Commit message: Updated damping and PID values for extension joints

File: dyret_description/urdf/dyret.xacro (robot description, xacro)
@@ -12,7 +12,7 @@
 		<plugin name="controller" filename="libdyret_gazebo_plugin.so">
 			<updateRate>50</updateRate>
-			<pid>1000.0 0.0 0</pid>
-			<pid type="mx64">8.6 0.5 1.0</pid>
-			<pid type="mx106">3.2 0.5 1.0</pid>
+			<pid>10000.0 0.0 100.0</pid>
+			<pid type="mx64">20 0.5 1.0</pid>
+			<pid type="mx106">20 0.5 1.0</pid>
 		</plugin>
 	</gazebo>

File: dyret_description/urdf/joints/large_extend.urdf.xacro (robot description, xacro)
@@ -57,5 +57,5 @@
 				lower="-0.100" upper="0.0"
 				effort="100.0" velocity="0.00045" />
-			<!--<dynamics damping="0.7" friction="0.1" />-->
+			<dynamics damping="200" friction="80" />
 		</joint>
 		<gazebo reference="${name}">

File: dyret_description/urdf/joints/small_extend.urdf.xacro (robot description, xacro)
@@ -57,5 +57,5 @@
 				lower="-0.025" upper="0.0"
 				effort="100.0" velocity="0.00045" />
-			<dynamics damping="0.7" friction="0.1" />
+			<dynamics damping="200" friction="80" />
 		</joint>
 		<gazebo reference="${name}">

Commit message: Updated PID and friction for extension joints

File: dyret_description/urdf/dyret.xacro (robot description, xacro)
@@ -12,5 +12,5 @@
 		<plugin name="controller" filename="libdyret_gazebo_plugin.so">
 			<updateRate>50</updateRate>
-			<pid>10000.0 0.0 100.0</pid>
+			<pid>20000.0 0.0 100.0</pid>
 			<pid type="mx64">20 0.5 1.0</pid>
 			<pid type="mx106">20 0.5 1.0</pid>

File: dyret_description/urdf/joints/large_extend.urdf.xacro (robot description, xacro)
@@ -61,5 +61,5 @@
 				lower="-0.100" upper="0.0"
 				effort="100.0" velocity="0.00045" />
-			<!--<dynamics damping="1.0" friction="80" />-->
+			<dynamics damping="1.0" friction="80" />
 		</joint>
 		<gazebo reference="${name}">
