Commit message: Added color to IMU and foot
Foot color is only enabled when using contact sensor to distinguish the
look and give visual feedback. The same is true for IMU, however, since
it is enabled by default it is expected that users will always see the
orange color.

File: dyret_description/urdf/imu.urdf.xacro (robot description, xacro)
@@ -25,4 +25,5 @@
 		<xacro:if value="$(arg imu_enabled)">
 			<gazebo reference="imu_link">
+				<material>Gazebo/Orange</material>
 				<gravity>true</gravity>
 				<sensor name="imu_sensor" type="imu">

File: dyret_description/urdf/joints/foot.urdf.xacro (robot description, xacro)
@@ -39,4 +39,5 @@
 				<maxVel>1.0</maxVel>
 				<minDepth>0.0</minDepth>
+				<material>Gazebo/Black</material>
 				<sensor name="${name}_bumper" type="contact">
 					<contact>
