Commit message: First commit with extended legs

File: dyret_description/urdf/dyret.urdf.xacro (robot description, xacro)
@@ -1,60 +1,41 @@
 <?xml version="1.0"?>
-<robot xmlns:xacro="http:/ros.org/wiki/xacro">
+<robot xmlns:xacro="http://ros.org/wiki/xacro">
 	<!-- Import complex parts for robot -->
-	<xacro:include filename="$(find dyret_description)/urdf/imu.urdf.xacro" />
+	<xacro:include filename="$(find dyret_description)/urdf/body.urdf.xacro" />
 	<xacro:include filename="$(find dyret_description)/urdf/leg.urdf.xacro" />
-	<!-- Leg to baseplate macro: -->
-	<xacro:macro name="base_leg" params="name rev frev">
-		<xacro:leg name="${name}" frev="${frev}"/>
-		<joint name="${name}_coxa_joint" type="revolute">
-			<origin xyz="${rev *(0.22 / 2 + 0.0208)} ${frev * (0.42 / 2 - 0.0058)} -0.0391"
-				rpy="0 1.57 0"/>
-			<parent link="baseplate" />
-			<child link="${name}_coxa" />
-			<dynamics damping="0.01" />
-			<limit effort="6.0" lower="-1.92" upper="1.92" velocity="2.57"/>
-			<axis xyz="0 1 0" />
+	<xacro:macro name="dyret_robot">
+		<xacro:body name="main_body" />
+		<xacro:leg name="fl" />
+		<joint name="fl_body_fixed" type="fixed">
+			<parent link="main_body_chassis" />
+			<child link="fl_joint1_servo" />
+			<origin xyz="${-body_width / 2 + mx64at_width/2 - 0.007}
+				${body_depth / 2 - mx64at_depth / 2 + 0.0065}
+				${-mx64at_height}" />
 		</joint>
-		<transmission name="${name}_coxa_transmission">
-			<type>transmission_interface/SimpleTransmission</type>
-			<actuator name="${name}_coxa_motor">
-				<hardwareInterface>hardware_interface/EffortJointInterface</hardwareInterface>
-				<mechanicalReduction>1</mechanicalReduction>
-			</actuator>
-			<joint name="${name}_coxa_joint">
-				<hardwareInterface>hardware_interface/EffortJointInterface</hardwareInterface>
-			</joint>
-		</transmission>
-	</xacro:macro>
-	<!-- Macro which builds the URDF -->
-	<xacro:macro name="dyret_robot">
-		<link name="baseplate">
-			<visual>
-				<geometry>
-					<mesh filename="package://dyret_description/meshes/base_assembly.STL" />
-				</geometry>
-			</visual>
-			<collision>
-				<geometry>
-					<box size="0.22 0.42 0.01" />
-				</geometry>
-			</collision>
-			<inertial>
-				<mass value="2.404" />
-				<inertia
-					ixx="0.035359" ixy="0.0" ixz="0.0"
-					iyy="0.009716" iyz="0.0"
-					izz="0.045035" />
-			</inertial>
-		</link>
-		<!-- Create four legs -->
-		<xacro:base_leg name="front_right" rev="1" frev="1" />
-		<xacro:base_leg name="front_left" rev="-1" frev="1" />
-		<xacro:base_leg name="back_right" rev="1" frev="-1" />
-		<xacro:base_leg name="back_left" rev="-1" frev="-1" />
-		<!-- Include IMU if desired -->
-		<xacro:if value="$(arg imu_enabled)">
-			<xacro:imu />
-		</xacro:if>
+		<xacro:leg name="fr" />
+		<joint name="fr_body_fixed" type="fixed">
+			<parent link="main_body_chassis" />
+			<child link="fr_joint1_servo" />
+			<origin xyz="${body_width / 2 - mx64at_width/2 + 0.012}
+				${body_depth / 2 - mx64at_depth / 2 + 0.005}
+				${-mx64at_height}" />
+		</joint>
+		<xacro:leg name="bl" />
+		<joint name="bl_body_fixed" type="fixed">
+			<parent link="main_body_chassis" />
+			<child link="bl_joint1_servo" />
+			<origin xyz="${-body_width / 2 + mx64at_width/2 - 0.01}
+				${-body_depth / 2 + mx64at_depth / 2 - 0.0035}
+				${-mx64at_height}" />
+		</joint>
+		<xacro:leg name="br" />
+		<joint name="br_body_fixed" type="fixed">
+			<parent link="main_body_chassis" />
+			<child link="br_joint1_servo" />
+			<origin xyz="${body_width / 2 - mx64at_width/2 + 0.009}
+				${-body_depth / 2 + mx64at_depth / 2 - 0.005}
+				${-mx64at_height}" />
+		</joint>
 	</xacro:macro>
 </robot>

File: dyret_description/urdf/dyret.xacro (robot description, xacro)
@@ -1,4 +1,4 @@
 <?xml version="1.0"?>
-<robot name="dyret" xmlns:xacro="http:/ros.org/wiki/xacro">
+<robot name="dyret" xmlns:xacro="http://ros.org/wiki/xacro">
 	<!-- Arguments that can be passed to this URDF file: -->
 	<xacro:arg name="imu_enabled" default="false" />

File: dyret_description/urdf/imu.urdf.xacro (robot description, xacro)
@@ -1,7 +1,8 @@
 <?xml version="1.0"?>
-<robot xmlns:xacro="http:/ros.org/wiki/xacro">
+<robot xmlns:xacro="http://ros.org/wiki/xacro">
+	<xacro:include filename="$(find dyret_description)/urdf/inertias.urdf.xacro" />
 	<!-- Macro for IMU -->
 	<xacro:macro name="imu">
-		<link name="imu">
+		<link name="imu_link">
 			<visual>
 				<origin xyz="0 0.003 0" rpy="0 0 3.1415" />
@@ -17,26 +18,30 @@
 				</geometry>
 			</collision>
-			<inertial>
-				<origin xyz="0 0 0.01" />
-				<mass value="0.052" />
-				<inertia
-					ixx="1.95e-05" ixy="0.0" ixz="0.0"
-					iyy="2.92e-05" iyz="0.0"
-					izz="2.92e-05" />
-			</inertial>
+			<xacro:box_inertia mass="0.052" width="0.057"
+				length="0.042" height="0.0235" r="${pi/2}"
+				y="${pi/2}"/>
 		</link>
-		<joint name="imu_joint" type="fixed">
-			<origin xyz="0 0 0"/>
-			<parent link="baseplate" />
-			<child link="imu" />
-		</joint>
-		<gazebo reference="imu">
-			<sensor name="imu_sensor" type="imu">
-				<always_on>true</always_on>
-				<update_rate>100</update_rate>
-				<visualize>true</visualize>
-				<topic>imu</topic>
-			</sensor>
-		</gazebo>
+		<!-- IMU Gazebo plugin support: -->
+		<xacro:if value="$(arg imu_enabled)">
+			<gazebo reference="imu_link">
+				<gravity>true</gravity>
+				<sensor name="imu_sensor" type="imu">
+					<always_on>true</always_on>
+					<update_rate>100</update_rate>
+					<visualize>true</visualize>
+					<topic>imu</topic>
+					<plugin filename="libgazebo_ros_imu_sensor.so" name="imu_plugin">
+						<bodyName>imu_link</bodyName>
+						<frameName>dyret_body</frameName>
+						<gaussianNoise>0.05</gaussianNoise>
+						<rpyOffset>0 0 0</rpyOffset>
+						<topicName>dyret/imu</topicName>
+						<updateRateHZ>100.0</updateRateHZ>
+						<xyzOffset>0 0 0</xyzOffset>
+					</plugin>
+					<pose>0 0 0 0 0 0</pose>
+				</sensor>
+			</gazebo>
+		</xacro:if>
 	</xacro:macro>
 </robot>

File: dyret_description/urdf/leg.urdf.xacro (robot description, xacro)
@@ -1,149 +1,44 @@
 <?xml version="1.0"?>
-<robot xmlns:xacro="http:/ros.org/wiki/xacro">
+<robot xmlns:xacro="http://ros.org/wiki/xacro">
+	<xacro:include filename="$(find dyret_description)/urdf/joints/mx106.urdf.xacro" />
+	<xacro:include filename="$(find dyret_description)/urdf/joints/mx64at.urdf.xacro" />
+	<xacro:include filename="$(find dyret_description)/urdf/joints/small_extend.urdf.xacro" />
+	<xacro:include filename="$(find dyret_description)/urdf/joints/large_extend.urdf.xacro" />
+	<xacro:include filename="$(find dyret_description)/urdf/joints/foot.urdf.xacro" />
 	<!-- Macro for one leg of Dyret -->
-	<xacro:macro name="leg" params="name frev">
-		<link name="${name}_coxa">
-			<visual>
-				<origin xyz="0.036 0 0" />
-				<geometry>
-					<mesh filename="package://dyret_description/meshes/coxa_assembly.STL" />
-				</geometry>
-			</visual>
-			<collision>
-				<origin xyz="0.036 0 0" />
-				<geometry>
-					<box size="0.072 0.051 0.051" />
-				</geometry>
-			</collision>
-			<inertial>
-				<origin xyz="0.036 0 0" />
-				<mass value="0.045" />
-				<inertia
-					ixx="1.95e-05" ixy="0.0" ixz="0.0"
-					iyy="2.92e-05" iyz="0.0"
-					izz="2.92e-05" />
-			</inertial>
-		</link>
-		<link name="${name}_femur">
-			<visual>
-				<origin xyz="0.0525 0 0" />
-				<geometry>
-					<mesh filename="package://dyret_description/meshes/femur_assembly.STL" />
-				</geometry>
-			</visual>
-			<collision>
-				<origin xyz="0.0525 0 0" />
-				<geometry>
-					<box size="0.129 0.0382 0.0503" />
-				</geometry>
-			</collision>
-			<inertial>
-				<origin xyz="0.0525 0 0" />
-				<mass value="0.3" />
-				<inertia
-					ixx="9.97e-05" ixy="0.0" ixz="0.0"
-					iyy="4.52e-04" iyz="0.0"
-					izz="4.79e-04" />
-			</inertial>
-		</link>
-		<joint name="${name}_femur_joint" type="revolute">
-			<origin xyz="0.072 0 0" rpy="0 0 ${frev * -1.047}" />
-			<parent link="${name}_coxa" />
-			<child link="${name}_femur" />
-			<!--<dynamics damping="0.01" />-->
-			<limit effort="6.0" lower="-1.92" upper="1.92" velocity="2.57" />
-			<axis xyz="0 0 1" />
+	<xacro:macro name="leg" params="name">
+		<xacro:mx64at_fr05h101 name="${name}_joint1"/>
+		<xacro:mx106t_fr08h101 name="${name}_joint2"/>
+		<joint name="${name}_joint1_2_fixed" type="fixed">
+			<parent link="${name}_joint1_bracket" />
+			<child link="${name}_joint2_bracket" />
+			<origin xyz="0 0 ${-mx64at_height/2 - fr05h101_height - 0.001}"
+				rpy="0 0 ${pi/2}" />
 		</joint>
-		<transmission name="${name}_femur_transmission">
-			<type>transmission_interface/SimpleTransmission</type>
-			<actuator name="${name}_femur_motor">
-				<hardwareInterface>hardware_interface/EffortJointInterface</hardwareInterface>
-				<mechanicalReduction>1</mechanicalReduction>
-			</actuator>
-			<joint name="${name}_femur_joint">
-				<hardwareInterface>hardware_interface/EffortJointInterface</hardwareInterface>
-			</joint>
-		</transmission>
-		<link name="${name}_tibia">
-			<visual>
-				<geometry>
-					<mesh filename="package://dyret_description/meshes/tibia_assembly.STL" />
-				</geometry>
-			</visual>
-			<!-- Collision element for servo bracket -->
-			<collision>
-				<origin xyz="0.018 0 0 " />
-				<geometry>
-					<box size="0.036 0.03 0.051" />
-				</geometry>
-			</collision>
-			<!-- Collision element for 3D printed holder -->
-			<collision>
-				<origin xyz="${0.06 + 0.036} 0 0 " />
-				<geometry>
-					<box size="0.12 0.03 0.0245" />
-				</geometry>
-			</collision>
-			<!-- Collision element for aluminium arm -->
-			<collision>
-				<origin xyz="${0.06 + 0.036 + 0.105} -0.0015 0 " />
-				<geometry>
-					<box size="0.098 0.012 0.012" />
-				</geometry>
-			</collision>
-			<!-- Collision element for rubber sphere -->
-			<collision>
-				<origin xyz="${0.06 + 0.036 + 0.105 + 0.053} -0.0015 0 " />
-				<geometry>
-					<sphere radius="0.01" />
-				</geometry>
-			</collision>
-			<inertial>
-				<origin xyz="0.15 0 0" />
-				<mass value="0.209" />
-				<inertia
-					ixx="2.61e-05" ixy="0.0" ixz="0.0"
-					iyy="9.21e-04" iyz="0.0"
-					izz="9.15e-04" />
-			</inertial>
-		</link>
-		<joint name="${name}_tibia_joint" type="revolute">
-			<origin xyz="0.1045 0 0" rpy="0 0 ${frev * 1.222}"/>
-			<parent link="${name}_femur" />
-			<child link="${name}_tibia" />
-			<!--<dynamics damping="0.01" />-->
-			<limit effort="6.0" lower="-1.92" upper="1.92" velocity="2.57" />
-			<axis xyz="0 0 1" />
+		<xacro:small_extender name="${name}_ext1" />
+		<joint name="${name}_joint2_ext1_fixed" type="fixed">
+			<parent link="${name}_joint2_servo" />
+			<child link="${name}_ext1_inner" />
+			<origin xyz="0 0 ${-mx106t_height/2 - fr08h101_height - small_ext_height/2}" />
 		</joint>
-		<transmission name="${name}_tibia_transmission">
-			<type>transmission_interface/SimpleTransmission</type>
-			<actuator name="${name}_tibia_motor">
-				<hardwareInterface>hardware_interface/EffortJointInterface</hardwareInterface>
-				<mechanicalReduction>1</mechanicalReduction>
-			</actuator>
-			<joint name="${name}_tibia_joint">
-				<hardwareInterface>hardware_interface/EffortJointInterface</hardwareInterface>
-			</joint>
-		</transmission>
-		<!-- This enables friction within Gazebo -->
-		<gazebo reference="${name}_tibia">
-			<mu1 value="200" />
-			<mu2 value="200" />
-			<!-- Include Contact sensor for feet -->
-			<xacro:if value="$(arg contact_enabled)">
-				<sensor name="${name}_contact_sensor" type="contact" always_on="true"
-					update_rate="10.0">
-					<contact>
-						<collision name="${name}_tibia_collision_3" />
-					</contact>
-					<plugin name="${name}_contact_plugin" filename="libgazebo_ros_bumper.so">
-						<alwaysOn>true</alwaysOn>
-						<updateRate>10.0</updateRate>
-						<frameName>world</frameName>
-						<bumperTopicName>${name}_contact</bumperTopicName>
-					</plugin>
-				</sensor>
-			</xacro:if>
-		</gazebo>
+		<xacro:mx106t_fr08h101_inv name="${name}_joint3" />
+		<joint name="${name}_ext1_joint3_fixed" type="fixed">
+			<parent link="${name}_ext1_outer" />
+			<child link="${name}_joint3_servo" />
+			<origin xyz="0 0.002 ${-small_ext_height/2 - small_ext2_height - mx106t_height/2}"
+				rpy="0 0 ${-pi/2}" />
+		</joint>
+		<xacro:large_extender name="${name}_ext2" />
+		<joint name="${name}_joint3_ext2_fixed" type="fixed">
+			<parent link="${name}_joint3_bracket" />
+			<child link="${name}_ext2_inner" />
+			<origin xyz="0 0 ${-fr08h101_height - large_ext_height + 0.0145/2}" />
+		</joint>
+		<xacro:foot name="${name}" />
+		<joint name="${name}_ext2_foot_fixed" type="fixed">
+			<parent link="${name}_ext2_outer" />
+			<child link="${name}_foot_cyl" />
+			<origin xyz="0 0 ${-large_ext2_height - 0.0355/2}" />
+		</joint>
 	</xacro:macro>
 </robot>

Commit message: Added external motor for extension joints and meshes

File: dyret_description/urdf/dyret.urdf.xacro (robot description, xacro)
@@ -14,5 +14,5 @@
 				${-mx64at_height}" />
 		</joint>
-		<xacro:leg name="fr" />
+		<xacro:leg name="fr" rot="-1" />
 		<joint name="fr_body_fixed" type="fixed">
 			<parent link="main_body_chassis" />
@@ -30,5 +30,5 @@
 				${-mx64at_height}" />
 		</joint>
-		<xacro:leg name="br" />
+		<xacro:leg name="br" rot="-1" />
 		<joint name="br_body_fixed" type="fixed">
 			<parent link="main_body_chassis" />

File: dyret_description/urdf/joints/foot.urdf.xacro (robot description, xacro)
@@ -4,9 +4,4 @@
 	<xacro:macro name="foot" params="name">
 		<link name="${name}_foot_cyl">
-			<visual>
-				<geometry>
-					<cylinder radius="0.014" length="0.0355" />
-				</geometry>
-			</visual>
 			<collision>
 				<geometry>

File: dyret_description/urdf/joints/large_extend.urdf.xacro (robot description, xacro)
@@ -27,10 +27,14 @@
 		</link>
 	</xacro:macro>
-	<xacro:macro name="large_ext2" params="name">
+	<xacro:macro name="large_ext2" params="name rot:=1">
 		<link name="${name}">
 			<visual>
-				<origin xyz="0 0 ${-large_ext2_height/2}" />
+				<origin rpy="0 0 ${pi/2 * rot}"
+					xyz="${(large_ext2_width * 2 - 0.009) * rot}
+					${(-large_ext2_depth * 2 - 0.002) * rot}
+					${-large_ext2_height * 1.5 + 0.005}" />
 				<geometry>
-					<box size="${large_ext2_width} ${large_ext2_depth} ${large_ext2_height}" />
+					<mesh filename="package://dyret_description/meshes/EXT2_OUTER.STL"
+						scale="0.001 0.001 0.001"/>
 				</geometry>
 			</visual>
@@ -46,7 +50,7 @@
 		</link>
 	</xacro:macro>
-	<xacro:macro name="large_extender" params="name">
+	<xacro:macro name="large_extender" params="name rot:=1">
 		<xacro:large_ext name="${name}_inner" />
-		<xacro:large_ext2 name="${name}_outer" />
+		<xacro:large_ext2 name="${name}_outer" rot="${rot}" />
 		<joint name="${name}" type="prismatic">
 			<parent link="${name}_inner" />
@@ -57,5 +61,5 @@
 				lower="-0.100" upper="0.0"
 				effort="100.0" velocity="0.00045" />
-			<dynamics damping="200" friction="80" />
+			<!--<dynamics damping="1.0" friction="80" />-->
 		</joint>
 		<gazebo reference="${name}">

File: dyret_description/urdf/joints/small_extend.urdf.xacro (robot description, xacro)
@@ -27,10 +27,12 @@
 		</link>
 	</xacro:macro>
-	<xacro:macro name="small_ext2" params="name">
+	<xacro:macro name="small_ext2" params="name rot:=1">
 		<link name="${name}">
 			<visual>
-				<origin xyz="0 0 ${-small_ext2_height/2}" />
+				<origin rpy="0 0 ${pi/2 * rot}"
+					xyz="${small_ext2_width/2 * rot} ${-small_ext2_depth/2 * rot} ${-small_ext2_height + 0.005}" />
 				<geometry>
-					<box size="${small_ext2_width} ${small_ext2_depth} ${small_ext2_height}" />
+					<mesh filename="package://dyret_description/meshes/EXT_OUTER.STL"
+						scale="0.001 0.001 0.001"/>
 				</geometry>
 			</visual>
@@ -46,7 +48,7 @@
 		</link>
 	</xacro:macro>
-	<xacro:macro name="small_extender" params="name">
+	<xacro:macro name="small_extender" params="name rot:=1">
 		<xacro:small_ext name="${name}_inner" />
-		<xacro:small_ext2 name="${name}_outer" />
+		<xacro:small_ext2 name="${name}_outer" rot="${rot}" />
 		<joint name="${name}" type="prismatic">
 			<parent link="${name}_inner" />
@@ -57,5 +59,5 @@
 				lower="-0.025" upper="0.0"
 				effort="100.0" velocity="0.00045" />
-			<dynamics damping="200" friction="80" />
+			<dynamics damping="1.0" friction="80" />
 		</joint>
 		<gazebo reference="${name}">

File: dyret_description/urdf/leg.urdf.xacro (robot description, xacro)
@@ -1,11 +1,12 @@
 <?xml version="1.0"?>
 <robot xmlns:xacro="http://ros.org/wiki/xacro">
+	<xacro:include filename="$(find dyret_description)/urdf/ext_motor.urdf.xacro" />
+	<xacro:include filename="$(find dyret_description)/urdf/joints/foot.urdf.xacro" />
+	<xacro:include filename="$(find dyret_description)/urdf/joints/large_extend.urdf.xacro" />
 	<xacro:include filename="$(find dyret_description)/urdf/joints/mx106.urdf.xacro" />
 	<xacro:include filename="$(find dyret_description)/urdf/joints/mx64at.urdf.xacro" />
 	<xacro:include filename="$(find dyret_description)/urdf/joints/small_extend.urdf.xacro" />
-	<xacro:include filename="$(find dyret_description)/urdf/joints/large_extend.urdf.xacro" />
-	<xacro:include filename="$(find dyret_description)/urdf/joints/foot.urdf.xacro" />
 	<!-- Macro for one leg of Dyret -->
-	<xacro:macro name="leg" params="name">
+	<xacro:macro name="leg" params="name rot:=1">
 		<xacro:mx64at_fr05h101 name="${name}_joint1"/>
 		<xacro:mx106t_fr08h101 name="${name}_joint2"/>
@@ -16,5 +17,11 @@
 				rpy="0 0 ${pi/2}" />
 		</joint>
-		<xacro:small_extender name="${name}_ext1" />
+		<xacro:ext_motor_upper name="${name}_ext_upper" rot="${rot}" />
+		<joint name="${name}_joint2_motor" type="fixed">
+			<parent link="${name}_joint2_servo" />
+			<child link="${name}_ext_upper" />
+			<origin xyz="${(-mx106t_width + 0.004) * rot} 0 ${-mx106t_height - 0.0395}" />
+		</joint>
+		<xacro:small_extender name="${name}_ext1" rot="${rot}" />
 		<joint name="${name}_joint2_ext1_fixed" type="fixed">
 			<parent link="${name}_joint2_servo" />
@@ -29,5 +36,11 @@
 				rpy="0 0 ${-pi/2}" />
 		</joint>
-		<xacro:large_extender name="${name}_ext2" />
+		<xacro:ext_motor_lower name="${name}_ext_lower" rot="${rot}" />
+		<joint name="${name}_joint3_motor" type="fixed">
+			<parent link="${name}_joint3_bracket" />
+			<child link="${name}_ext_lower" />
+			<origin xyz="${(-fr08h101_width + 0.008) * rot} ${0.001 * rot} ${-fr08h101_height * 2 - 0.003}" />
+		</joint>
+		<xacro:large_extender name="${name}_ext2" rot="${rot}" />
 		<joint name="${name}_joint3_ext2_fixed" type="fixed">
 			<parent link="${name}_joint3_bracket" />
