Commit message: Updated height of extension joint 1

File: dyret_description/urdf/joints/large_extend.urdf.xacro (robot description, xacro)
@@ -61,5 +61,5 @@
 				lower="-0.100" upper="0.0"
 				effort="100.0" velocity="0.00045" />
-			<dynamics damping="1.0" friction="80" />
+			<dynamics damping="1.0" friction="70" />
 		</joint>
 		<gazebo reference="${name}">

File: dyret_description/urdf/joints/small_extend.urdf.xacro (robot description, xacro)
@@ -7,5 +7,5 @@
 	<xacro:property name="small_ext2_width" value="0.0436" />
 	<xacro:property name="small_ext2_depth" value="0.0212" />
-	<xacro:property name="small_ext2_height" value="0.0792" />
+	<xacro:property name="small_ext2_height" value="0.06" />
 	<xacro:macro name="small_ext" params="name">
 		<link name="${name}">
